File: FINAL TASK/Finale.kicad_pcb (KiCad board)
At the start: 2 copper layers, 36 parts, among them J1 Conn_01x04_Pin, J2 Conn_01x04_Pin, P1 USB_C_Plug, SW1 RESET, SW2 SW_SPDT, U1 STM32F103C8T6, U2 AS5048B, U3 AS5048B, U4 AS5048B, U5 AS5048B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

Commit message: C
Parts:
- removed C17, C18: 1uF, Capacitor_SMD:C_0402_1005Metric
- removed D1: D, Diode_SMD:D_0805_2012Metric
- removed FB1: FerriteBead, Inductor_SMD:L_0805_2012Metric
- removed R1, R2: 27, Resistor_SMD:R_0805_2012Metric
- added C15: 100nF, Capacitor_SMD:C_0402_1005Metric, F.Cu at (155.9, 91.3)
- C10, C11, C12, C13, C9: footprint Capacitor_SMD:C_0805_2012Metric -> Capacitor_SMD:C_0402_1005Metric
- C14: value 10nF -> 100nF
- P1: footprint Connector_USB:USB_C_Plug_Molex_105444 -> USB-C:GCT_USB4085-GF-A_REVB
- SW1: footprint Button_Switch_SMD:SW_Push_SPST_NO_Alps_SKRK -> SPST:SW_FSM8JH
- SW2: footprint Button_Switch_SMD:SW_SPDT_CK_JS102011SAQN -> SPDT:SW_MINI-SPDT-SW
- moved C1 140.1 mm to (184.2, 99.8), turned to 90 degrees
- moved SW1 139.3 mm to (177.6, 103.3), turned to 90 degrees
- moved C13 124.6 mm to (185.6, 88.2)
- moved C8 117.2 mm to (167.8, 99.4)
- moved C11 113.8 mm to (170.5, 91.8), turned to -90 degrees
- moved U5 112.0 mm to (143.0, 103.6)
- moved U4 111.2 mm to (143.0, 95.5)
- moved R3 110.8 mm to (171.7, 101.5), turned to -90 degrees
- moved U3 110.3 mm to (143.0, 87.4)
- moved U2 109.4 mm to (143.1, 78.9)
- moved U6 108.8 mm to (180.0, 93.2)
- moved SW2 104.7 mm to (158.3, 105.5)
- moved C10 99.5 mm to (147.6, 102.5), turned to 90 degrees
- moved R4 98.7 mm to (159.3, 102.0)
- moved C9 93.1 mm to (147.6, 86.5), turned to 90 degrees
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Connections:
- C14 pad 1: +3.3VA -> +3.3V
- P1 pad A6: Net-(P1-D+) -> /DP
- P1 pad A7: Net-(P1-D-) -> /DM
- P1 pad S1: unconnected-(P1-SHIELD-PadS1) -> GND
- U1 pad 1: unconnected-(U1B-VBAT-Pad1) -> +3.3V
- U1 pad 9: +3.3VA -> +3.3V
- U2 pad 5: unconnected-(U2-TEST-Pad5) -> GND
- U3 pad 5: unconnected-(U3-TEST-Pad5) -> GND
- U4 pad 5: unconnected-(U4-TEST-Pad5) -> GND
- U5 pad 5: unconnected-(U5-TEST-Pad5) -> GND
Routing:
- net +3.3V: track 0.00 -> 201.1 mm, vias 0 -> 2
- net /I2C_SDA: track 0.00 -> 80.9 mm, vias 0 -> 2
- net /I2C_SCL: track 0.00 -> 75.5 mm, vias 0 -> 6
- net GND: track 0.00 -> 62.3 mm, vias 0 -> 19
- net /RST: track 0.00 -> 31.2 mm
- net VBUS: track 0.00 -> 27.8 mm
- net /DM: track 0.00 -> 27.7 mm, vias 0 -> 1
- net /SWCLK: track 0.00 -> 25.3 mm, vias 0 -> 2
- net /SWDIO: track 0.00 -> 24.2 mm, vias 0 -> 1
- net /DP: track 0.00 -> 23.2 mm
- net /BOOT: track 0.00 -> 13.4 mm, vias 0 -> 2
- net /OSC_IN: track 0.00 -> 8.17 mm
- net /OSC_OUT: track 0.00 -> 5.64 mm
- net Net-(SW2-B): track 0.00 -> 3.49 mm
- added copper zone on B.Cu, net GND
Other:
- board outline added: 58.2 x 41.1 mm

Commit message: Done
Parts:
- added H1: MountingHole, MountingHole:MountingHole_2.1mm, F.Cu at (138.0, 72.2)
- added H2: MountingHole, MountingHole:MountingHole_2.1mm, F.Cu at (192.8, 71.7)
- added H3: MountingHole, MountingHole:MountingHole_2.1mm, F.Cu at (193.0, 108.2)
- added H4: MountingHole, MountingHole:MountingHole_2.1mm, F.Cu at (137.3, 108.0)
- moved R5 5.47 mm to (149.6, 81.7), turned to 90 degrees
- moved P1 3.52 mm to (194.1, 92.3)
- moved U5 1.17 mm to (143.0, 102.4)
- moved C13 0.30 mm to (185.3, 88.1)
- moved Y1 0.11 mm to (151.9, 93.6)
Routing:
- net +3.3V: track 201.1 -> 289.8 mm, vias 2 -> 5
- net VBUS: track 27.8 -> 34.5 mm
- net /I2C_SCL: track 75.5 -> 69.7 mm
- net /DP: track 23.2 -> 27.0 mm
- net /DM: track 27.7 -> 31.5 mm
- net GND: track 62.3 -> 64.4 mm, vias 19 -> 17
- net /I2C_SDA: track 80.9 -> 79.3 mm
- net /OSC_IN: track 8.17 -> 7.67 mm
Other:
- board size 58.2 x 41.1 mm -> 61.4 x 42.3 mm
- board text added: "U2"
